File: nicklink.kicad_pcb (KiCad board)
At the start: 2 copper layers, 34 x 33 mm, 34 parts, among them J1 Conn_02x10_Odd_Even, J2 USB_C_Receptacle_USB2.0_16P, J3 Conn_02x10_Odd_Even, SW1 SW_SPDT, U1 STM32F103C8T6, U2 AMS1117-3.3, Y1 16MHz

Commit message: Polish public repo: MIT license, nicklink naming, docs sync
Add MIT LICENSE, rename pcb_hello_world footprints/fab files to nicklink,
align README area claim with REVIEW (49.7%), and fix REVIEW paths to match
what this repository actually ships.
Parts:
- J2: footprint pcb_hello_world:USB_C_Receptacle_GCT_USB4085_EdgeSilk -> nicklink:USB_C_Receptacle_GCT_USB4085_EdgeSilk
- SW1: footprint pcb_hello_world:SW_SPDT_PCM12_EdgeSilk -> nicklink:SW_SPDT_PCM12_EdgeSilk
Changed lines of the file:
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@@
 		)
 	)
-	(footprint "pcb_hello_world:SW_SPDT_PCM12_EdgeSilk"
+	(footprint "nicklink:SW_SPDT_PCM12_EdgeSilk"
 		(layer "F.Cu")
 		(at 104 62.8 180)
@@
 		)
 	)
-	(footprint "pcb_hello_world:USB_C_Receptacle_GCT_USB4085_EdgeSilk"
+	(footprint "nicklink:USB_C_Receptacle_GCT_USB4085_EdgeSilk"
 		(layer "F.Cu")
 		(at 97.175 66.625 180)
