File: nicklink.kicad_sch (KiCad schematic)
At the start: 30 parts, among them J1 Conn_02x10_Odd_Even, J2 USB_C_Receptacle_USB2.0_16P, J3 Conn_02x10_Odd_Even, SW1 SW_SPDT, U1 STM32F103C8T6, U2 AMS1117-3.3, Y1 16MHz

Commit message: NickLink v1.2 — smaller board, front pin labels, QoL fixes
Board shrinks from 34 x 33 mm to 33.19 x 25.5 mm (-25% area) while keeping
both 2x10 headers and all four M2 holes, and every header pin is now labelled
beside it on the front silkscreen.

Hardware changes:
- 5 V on J1.1 (USB VBUS via 1N5819WS Schottky; usable as a <=5.5 V input)
- RESET and BOOT buttons (B3U); NRST moved to J3 next to SWDIO/SWCLK/SWO
- 8 MHz HSE crystal (was 16 MHz), 15 pF load caps
- TLV75533 WSON LDO + ceramics replaces AMS1117 + tantalum
- USBLC6-2P6 ESD on D+/D-/VBUS
- I2C pull-ups on PB6/PB7 removed; user LED on PC13
- Header pinout reordered to follow the MCU package order

The design is now generated: tools/spec.py and tools/placement.py drive the
schematic, placement, Freerouting autoroute, GND stitching, DRC and fab
outputs (tools/build_all.sh, tools/fab.sh), all in Docker. ERC 0/0, DRC 0
violations / 0 unconnected / 0 parity issues.

Docs, renders, pinout CSV, schematic PDF, assembly/copper PDFs and
fabrication/v1.2 (Gerbers, drills, JLC BOM/CPL) are updated; v1.1 fab
outputs are kept.

Co-Authored-By: Claude Opus 5.5 <noreply@anthropic.com>
Claude-Session: https://claude.ai/code/session_01KPMtzubqGeBFaq48UcVZaf
Parts:
- removed C13: 22u tantalum, Capacitor_Tantalum_SMD:CP_EIA-3216-18_Kemet-A, symbol Device:C_Polarized
- removed R7: 1k5, Resistor_SMD:R_0402_1005Metric, symbol Device:R
- removed SW1: SW_SPDT, nicklink:SW_SPDT_PCM12_EdgeSilk, symbol Switch:SW_SPDT
- removed U2: AMS1117-3.3, Package_TO_SOT_SMD:SOT-223-3_TabPin2, symbol Regulator_Linear:AMS1117-3.3
- added C13: 100n, Capacitor_SMD:C_0402_1005Metric, symbol Device:C
- added D2: 1N5819WS, Diode_SMD:D_SOD-323, symbol Device:D_Schottky
- added D3: GREEN, LED_SMD:LED_0402_1005Metric, symbol Device:LED
- added SW1: RESET, nicklink:SW_SPST_B3U-1000P_NoSilk, symbol Switch:SW_Push
- added SW2: BOOT0, nicklink:SW_SPST_B3U-1000P_NoSilk, symbol Switch:SW_Push
- added U2: TLV75533PDRV, Package_SON:WSON-6-1EP_2x2mm_P0.65mm_EP1x1.6mm, symbol Regulator_Linear:TLV75533PDRV
- added U3: USBLC6-2P6, Package_TO_SOT_SMD:SOT-666, symbol Power_Protection:USBLC6-2P6
- C1: LCSC (none) -> C1525; Note (none) -> VDD pin 1/VBAT decoupling
- C10, C11: value 10p -> 15p; LCSC (none) -> C1548; Note (none) -> C0G; crystal CL 12 pF
- C12: value 4.7u -> 1u; footprint Capacitor_SMD:C_0805_2012Metric -> Capacitor_SMD:C_0402_1005Metric; LCSC (none) -> C52923; Note (none) -> LDO input
- C2: LCSC (none) -> C1525; Note (none) -> VDD pin 24 decoupling
- C3: LCSC (none) -> C1525; Note (none) -> VDD pin 36 decoupling
- C4: LCSC (none) -> C1525; Note (none) -> VDD pin 48 decoupling
- C5: LCSC (none) -> C19702; Note (none) -> 3V3 bulk
- C6: LCSC (none) -> C1525; Note (none) -> VDDA
- C7: LCSC (none) -> C52923; Note (none) -> VDDA
- C8: LCSC (none) -> C52923; Note (none) -> LDO output
- C9: LCSC (none) -> C1525
- D1: footprint LED_SMD:LED_0603_1608Metric -> LED_SMD:LED_0402_1005Metric; LCSC (none) -> C264407; MPN (none) -> Everlight 16-213/R6C-AQ2R2B/3T; Note (none) -> Power
- FB1: value 120R -> 120R@100MHz; footprint Inductor_SMD:L_0603_1608Metric -> Inductor_SMD:L_0402_1005Metric; LCSC (none) -> C85812
- J1, J3: footprint Connector_PinHeader_2.54mm:PinHeader_2x10_P2.54mm_Vertical -> nicklink:PinHeader_2x10_P2.54mm_Vertical_NoSilk
- J2: LCSC (none) -> C7095263; MPN (none) -> GCT USB4085-GF-A
- R1: LCSC (none) -> C25744; Note (none) -> BOOT0 pull-down
- R2: LCSC (none) -> C25867; Note (none) -> USB FS D+ pull-up
- R3, R6: LCSC (none) -> C25867
- R4, R5: LCSC (none) -> C25905
- R8: LCSC (none) -> C25744; Note (none) -> BOOT1 pull-down
- U1: LCSC (none) -> C8734
- Y1: value 16MHz -> 8MHz; LCSC (none) -> C2682775; MPN (none) -> YXC X32258MOB4SI (CL 12 pF)
Connections:
- net BOOT_SELECT is gone; now on net BOOT0: R1.1
- net +3.3V: now also J1.20 (Pin_20), D3.2 (A), SW2.1, U2.1 (OUT); no longer J1.1 (Pin_1), R6.1
- net BOOT0: now also SW2.2; no longer R1.2
- net GND: now also R1.2, C13.2, SW1.2, U2.3 (GND), U2.7 (GND), U3.2 (GND); no longer J1.20 (Pin_20)
- net NRST: now also J3.10 (Pin_10), SW1.1; no longer J1.6 (Pin_6)
- net PA0: now also J1.19 (Pin_19); no longer J1.7 (Pin_7)
- net PA1: now also J1.18 (Pin_18); no longer J1.8 (Pin_8)
- net PA15: now also J3.6 (Pin_6); no longer J3.10 (Pin_10)
- net PA2: now also J1.17 (Pin_17); no longer J1.9 (Pin_9)
- net PA3: now also J1.16 (Pin_16); no longer J1.10 (Pin_10)
- net PA4: now also J1.15 (Pin_15); no longer J1.11 (Pin_11)
- net PA8: now also J3.5 (Pin_5); no longer J3.15 (Pin_15)
- net PB0: now also J1.11 (Pin_11); no longer J1.15 (Pin_15)
- net PB1: now also J1.10 (Pin_10); no longer J1.16 (Pin_16)
- net PB10: now also J1.8 (Pin_8); no longer J1.18 (Pin_18)
- net PB11: now also J1.7 (Pin_7); no longer J1.19 (Pin_19)
- net PB12: now also J1.6 (Pin_6); no longer J3.19 (Pin_19)
- net PB13: now also J1.5 (Pin_5); no longer J3.18 (Pin_18)
- net PB14: now also J1.4 (Pin_4); no longer J3.17 (Pin_17)
- net PB15: now also J1.3 (Pin_3); no longer J3.16 (Pin_16)
- net PB2: now also J1.9 (Pin_9); no longer J1.17 (Pin_17)
- net PB4: now also J3.11 (Pin_11); no longer J3.8 (Pin_8)
- net PB5: now also J3.12 (Pin_12); no longer J3.7 (Pin_7)
- net PC13: now also J3.17 (Pin_17), R6.1; no longer J1.3 (Pin_3)
- net PC14: now also J3.18 (Pin_18); no longer J1.4 (Pin_4)
- net PC15: now also J3.19 (Pin_19); no longer J1.5 (Pin_5)
- net USB_D+: now also U3.1 (I/O1), U3.6 (I/O1)
- net USB_D-: now also U3.3 (I/O2), U3.4 (I/O2)
- net VBUS: now also C13.1, D2.2 (A), U3.5 (VBUS); no longer C12.1
- net CAN_RX renamed PA9
- net PA9: now also U1.30 (PA9); no longer U1.45 (PB8)
- net CAN_TX renamed PA10
- net PA10: now also U1.31 (PA10); no longer U1.46 (PB9)
- removed net I2C1_SCL: J3.5 (Pin_5), R6.2, U1.42 (PB6)
- net I2C1_SDA renamed PB7
- net PB7: now also J3.14 (Pin_14); no longer J3.6 (Pin_6)
- net SPI1_MISO renamed PA6
- net SPI1_MOSI renamed PA5
- net PA5: now also U1.15 (PA5); no longer U1.17 (PA7)
- net SPI1_SCK renamed PA7
- net PA7: now also U1.17 (PA7); no longer U1.15 (PA5)
- net SWCLK renamed PA14
- net PA14: now also J3.8 (Pin_8); no longer J3.11 (Pin_11)
- net SWDIO renamed PA13
- net PA13: now also J3.7 (Pin_7); no longer J3.12 (Pin_12)
- removed net USART1_RX: J3.14 (Pin_14), U1.31 (PA10)
- net USART1_TX renamed PB6
- net PB6: now also U1.42 (PB6); no longer U1.30 (PA9)
- new net +5V: C12.1, D2.1 (K), J1.1 (Pin_1), U2.4 (EN), U2.6 (IN)
- new net PB8: J3.15 (Pin_15), U1.45 (PB8)
- new net PB9: J3.16 (Pin_16), U1.46 (PB9)
- new net USER_LED_K: D3.1 (K), R6.2
Other:
- note added: "CLOCK (8 MHZ HSE)"
- note added: "HEADERS J1 / J3"
- note added: "MCU + DECOUPLING"
- note added: "NOTES 1. Every header pin is labelled beside it on the front silkscreen (A9 = PA9); the back has a function cheat sheet. 2. CAN (PB8 RX / PB9 TX, remapped) is logic level only: it needs an external CAN transceiver. 3. USB and CAN cannot run at the same time on the STM32F103 (they share the packet RAM). 4. The 3V3 header pins are outputs of the on-board LDO (U2); do not back-drive them from anothe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"
- note added: "POWER"
- note added: "RESET / BOOT"
- note added: "USB-C + ESD"
- note added: "USER LED"
- note removed: "3V3 pins are regulated outputs. Do not connect another powered 3V3 supply while USB is attached."
- note removed: "J1: GPIO / ADC / SPI / RESET"
- note removed: "J3: DEBUG / UART / I2C / CAN LOGIC"
- note removed: "Two identical 2x10 headers, 2.54 mm pitch. CAN pins require an external transceiver."
- title: (none) -> NickLink

Commit message: NickLink v1.3 — on-board 6-axis IMU (LSM6DSV16X)
Adds an ST LSM6DSV16X accel+gyro on I2C1 (PB6/PB7, address 0x6A) with
INT1 on PA0 (WKUP), for motion tracking, robotics and tap-to-wake use.
Placed on the top side (single-sided assembly): the board grows to
33.19 x 28.8 mm (956 mm^2, still -15% vs v1.1). Pinout unchanged from v1.2.

- 4.7k I2C1 pull-ups restored (on-board device on the bus)
- Project symbol nicklink:LSM6DSV16X; top-copper keep-out under the package
- Crystal nets pre-routed as locked top-layer tracks (no vias)
- USBLC6 channels swapped so D+/D- don't cross at the MCU
- Min track width 0.10 mm to accept Freerouting neck-downs
- build_pcb.py --resilk for silkscreen-only edits; build_all.sh retries
  autoroute; seeded placement search documented in tools/README.md
- README, design review, pinout CSV, schematic, PDFs, renders, checks and
  fabrication/v1.3 updated

ERC 0/0; DRC 0 violations, 0 unconnected, 0 parity issues.

Co-Authored-By: Claude Opus 5.5 <noreply@anthropic.com>
Claude-Session: https://claude.ai/code/session_01KPMtzubqGeBFaq48UcVZaf
Parts:
- added C14, C15: 100n, Capacitor_SMD:C_0402_1005Metric, symbol Device:C
- added R7, R9: 4k7, Resistor_SMD:R_0402_1005Metric, symbol Device:R
- added U4: LSM6DSV16X, nicklink:LGA-14_3x2.5mm_P0.5mm_LayoutBorder3x4y_NoSilk, symbol nicklink:LSM6DSV16X
Connections:
- net +3.3V: now also C14.1, C15.1, R7.1, R9.1, U4.12 (CS), U4.5 (VDDIO), U4.8 (VDD)
- net GND: now also C14.2, C15.2, U4.1 (SDO/SA0), U4.2 (SDX), U4.3 (SCX), U4.6 (GND), U4.7 (GND)
- net PA0: now also U4.4 (INT1)
- net PB6: now also R7.2, U4.13 (SCL)
- net PB7: now also R9.2, U4.14 (SDA)
- net USB_D+: now also U3.3 (I/O2), U3.4 (I/O2); no longer U3.1 (I/O1), U3.6 (I/O1)
- net USB_D-: now also U3.1 (I/O1), U3.6 (I/O1); no longer U3.3 (I/O2), U3.4 (I/O2)
- no-connect marks 2 -> 5
Other:
- note added: "IMU (I2C1 0X6A, INT1 -> PA0)"

Commit message: v1.3: fix the five-reviewer audit findings
Independent reviews (power, MCU, USB, IMU/headers, fab/DFM) found issues that
would have made the board fail or be unreliable. Fixed:

- CPL: per-footprint JLC rotation corrections (LQFP-48 -90, SOT-666 +180,
  LGA-14 +180), verified against JLC's EasyEDA footprints. As shipped, U1
  would have been rotated 90 deg and U3 would have shorted VBUS to GND.
- LDO: output cap C8 now 0.95 mm from OUT; C12 -> 10 uF 0603; two 0.3 mm
  thermal vias in the exposed pad (project WSON footprint).
- IMU INT1 (forced low at power-up) now reaches A0 through R10 10k.
- USB4085: 0.38 mm holes / 0.74 mm pads (inside GCT's 0.40 +-0.05 spec,
  JLC 0.18 mm ring), thermal-relief GND pins.
- IMU: no pour under the body, pre-routed local fan-out (GND vias, 3V3 rail,
  B.Cu GND link under the MCU); OCS_Aux/SDO_Aux tied to VDDIO.
- VDDA caps next to the VDDA pin; MCU group 0.25 mm left so fan-out vias fit.
- Docs: PB6/PB7 and NRST are 3.3 V only, I2C pull-ups to 3.3 V only, ENIG,
  hardware/back-feed notes; review summary in docs/REVIEW.md.
- Tooling: pour-only rule areas no longer exported as DSN keepouts; B.Cu
  pre-routes and pre-placed vias; stitching respects oval slots.

ERC 0/0; DRC 0 violations, 0 unconnected, 0 parity issues.

Co-Authored-By: Claude Opus 5.5 <noreply@anthropic.com>
Claude-Session: https://claude.ai/code/session_01KPMtzubqGeBFaq48UcVZaf
Parts:
- added R10: 10k, Resistor_SMD:R_0402_1005Metric, symbol Device:R
- C12: value 1u -> 10u; footprint Capacitor_SMD:C_0402_1005Metric -> Capacitor_SMD:C_0603_1608Metric; LCSC C52923 -> C19702; Note LDO input -> LDO input + VBUS hot-plug bulk (USB allows <= 10 uF)
- C14: Note IMU VDD -> IMU VDD/VDDIO
- C15: Note IMU VDDIO -> IMU VDD/VDDIO
- U2: footprint Package_SON:WSON-6-1EP_2x2mm_P0.65mm_EP1x1.6mm -> nicklink:WSON-6-1EP_2x2mm_P0.65mm_EP1x1.6mm_ThermalVias03
Connections:
- net +3.3V: now also U4.10 (OCS_Aux), U4.11 (SDO_Aux)
- net PA0: now also R10.2; no longer U4.4 (INT1)
- new net IMU_INT1: R10.1, U4.4 (INT1)
- no-connect marks 5 -> 3
Other:
- note added: "IMU (I2C1 0X6A, INT1 -> 10K -> PA0)"
- note removed: "IMU (I2C1 0X6A, INT1 -> PA0)"

Commit message: v1.3 reliability pass: protected power path, STM32 best practices, SPICE + emulated test firmware
Power: R12 1R anti-surge in series with VBUS (hot-plug ring 6.1-11.4 V -> 5.38 V
at LDO IN, inrush 33 uC); C12 4.7 uF, 3V3 10 uF bulk removed; F1 0.5 A PTC + Q1
DMP2165UW reverse-polarity FET on the J1.1 5V pin branch.
STM32: 4.7 uF on VDD3 (DS5319 Fig. 14); D+ pull-up from VBUS (R2 2k2 + R11 4k7,
AN4879 3.1.1) so J1.1 power no longer back-feeds the host; R6 330R user LED.
Layout: locked USB-C orientation ties, VBUS path U3 -> C13 -> J2, IMU GND return
via its caps, GND vias for R3/VSS_2; seed 12 baked, finished with the new
tools/fixroute.sh grid router. stitch.py checks connectivity per pour island
(tools/gndnet.py). DRC 0/0/0, ERC 0/0.
sim/: ngspice benches 1-11 (as-built table in results/summary.md).
firmware/: bare-metal bring-up firmware + Renode board model, 10 tests pass.

Co-Authored-By: Claude Opus 5.5 <noreply@anthropic.com>
Claude-Session: https://claude.ai/code/session_01KPMtzubqGeBFaq48UcVZaf
Parts:
- removed C5: 10u, Capacitor_SMD:C_0603_1608Metric, symbol Device:C
- added F1: 0.5A, Fuse:Fuse_0805_2012Metric, symbol Device:Polyfuse
- added Q1: DMP2165UW, nicklink:SOT-323_SC-70_NoSilk, symbol Transistor_FET:DMG2301L
- added R11: 4k7, nicklink:R_0402_1005Metric_NoSilk, symbol Device:R
- added R12: 1R, Resistor_SMD:R_0805_2012Metric, symbol Device:R
- C12: value 10u -> 4u7; footprint Capacitor_SMD:C_0603_1608Metric -> Capacitor_SMD:C_0402_1005Metric; LCSC C19702 -> C23733; Note LDO input + VBUS hot-plug bulk (USB allows <= 10 uF) -> LDO input (10 V X5R; USB allows <= 10 uF)
- C4: value 100n -> 4u7; LCSC C1525 -> C23733; Note VDD pin 48 decoupling -> VDD3 (pin 48) bulk: DS5319 Fig. 14 requires 4.7 uF on VDD3
- D2: Note Blocks back-feed from the 5V header pin into USB -> Blocks back-feed from VSYS / the 5V pin into USB
- R2: value 1k5 -> 2k2; LCSC C25867 -> C25879; Note USB FS D+ pull-up -> USB FS D+ pull-up (with R11: 1.5k to 3.4 V, VBUS-derived)
- R5, R8: footprint Resistor_SMD:R_0402_1005Metric -> nicklink:R_0402_1005Metric_NoSilk
- R6: value 1k5 -> 330; LCSC C25867 -> C25104; Note (none) -> ~1.2-1.8 mA (PC13 sinks <= 3 mA)
Connections:
- net +3.3V: no longer R2.1
- net +5V: now also Q1.3 (D); no longer C12.1, D2.1 (K), U2.4 (EN), U2.6 (IN)
- net GND: now also Q1.1 (G), R11.1
- net USB_D+: now also R11.2
- net VBUS: now also R2.1, R12.1; no longer D2.2 (A)
- new net 5V_F: F1.2, Q1.2 (S)
- new net VBUS_D: D2.2 (A), R12.2
- new net VSYS: C12.1, D2.1 (K), F1.1, U2.4 (EN), U2.6 (IN)

Commit message: v1.3 second review wave: TLV76733 LDO, VBUS_D off the USB shell, IMU spacing, firmware fixes
Five reviewers (power C+, MCU B, USB B, IMU/GPIO B+, fab B+); all must-fixes done:
- U2 TLV75533 -> TLV76733DRVR (same DRV0006A pads, VIN/EN 18 V): J1.1 hot-plug
  rang VSYS past the TLV755's 6 V abs max. SNS->OUT, pin 5->GND stubs. C12 16 V.
  New SPICE bench 12 (J1.1 hot-plug, 1.5-3 uH USB cables).
- VBUS_D hops to B.Cu under the USB4085 shell; F.Cu keep-out over its GND dimples.
- IMU: pour keep-out off the GND pads, bottom GND via outside the body.
- Net classes: signals 0.127/0.127 mm, GND and new Rail class (3V3) 0.2 mm; seed 3
  now routes 100% with Freerouting alone. DRC 0/0/0, ERC 0/0, one GND cluster,
  no via within 0.1 mm of an SMD pad.
- Tools: stitch.py keeps vias off SMD pads; fixroute.py via/screw keep-outs and
  path smoothing; autoroute RIPUP=1 second pass; swapfp.py.
- Firmware: VTOR, clock bring-up from any state, CSS/NMI fallback, PVD 2.9 V,
  standby (WKUP) and adc commands, pin-map test fixed: Renode 10/10.
- Docs: 5V-pin output/short behaviour, battery caveat, PC13-15 shared 3 mA,
  I2C1/SPI1 remap conflicts (ES096), review write-up in docs/REVIEW.md.

Co-Authored-By: Claude Opus 5.5 <noreply@anthropic.com>
Claude-Session: https://claude.ai/code/session_01KPMtzubqGeBFaq48UcVZaf
Parts:
- C12: value 4u7 -> 4u7 16V; LCSC C23733 -> C318563; MPN (none) -> Samsung CL05A475MO5NUNC; Note LDO input (10 V X5R; USB allows <= 10 uF) -> LDO input, 16 V X5R (J1.1 hot-plug ring); USB allows <= 10 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
- U2: value TLV75533PDRV -> TLV76733DRVR; symbol Regulator_Linear:TLV75533PDRV -> nicklink:TLV76733DRV; LCSC C2861750 -> C2848334; MPN (none) -> TI TLV76733DRVR
Connections:
- net +3.3V: now also U2.2 (SNS)
- net GND: now also U2.5 (GND)
Changed lines of the file:
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@@
           (size 1.27 1.27))
         (justify left)))
-    (property "Value" "4u7"
+    (property "Value" "4u7 16V"
       (at 313.182 41.91 0)
       (show_name no)
@@
         (font
           (size 1.27 1.27))))
-    (property "Note" "LDO input (10 V X5R; USB allows <= 10 uF)"
-      (at 309.88 40.64 0)
-      (hide yes)
-      (show_name no)
-      (do_not_autoplace no)
-      (effects
-        (font
-          (size 1.27 1.27))))
-    (property "LCSC" "C23733"
+    (property "Note" "LDO input, 16 V X5R (J1.1 hot-plug ring); USB allows <= 10 uF"
+      (at 309.88 40.64 0)
+      (hide yes)
+      (show_name no)
+      (do_not_autoplace no)
+      (effects
+        (font
+          (size 1.27 1.27))))
+    (property "MPN" "Samsung CL05A475MO5NUNC"
+      (at 309.88 40.64 0)
+      (hide yes)
+      (show_name no)
+      (do_not_autoplace no)
+      (effects
+        (font
+          (size 1.27 1.27))))
+    (property "LCSC" "C318563"
       (at 309.88 40.64 0)
       (hide yes)
@@
           (unit 1)))))
   (symbol
-    (lib_id "Regulator_Linear:TLV75533PDRV")
+    (lib_id "nicklink:TLV76733DRV")
     (at 335.28 40.64 0)
     (unit 1)
@@
         (font
           (size 1.27 1.27))))
-    (property "Value" "TLV75533PDRV"
+    (property "Value" "TLV76733DRVR"
       (at 335.28 34.925 0)
       (show_name no)
@@
         (font
           (size 1.27 1.27))))
-    (property "Datasheet" "http://www.ti.com/lit/ds/symlink/tlv755p.pdf"
-      (at 335.28 40.64 0)
-      (hide yes)
-      (show_name no)
-      (do_not_autoplace no)
-      (effects
-        (font
-          (size 1.27 1.27))))
-    (property "Description" "500mA Low Dropout Voltage Regulator, Fixed Output 3.3V, WSON6"
-      (at 335.28 40.64 0)
-      (hide yes)
-      (show_name no)
-      (do_not_autoplace no)
-      (effects
-        (font
-          (size 1.27 1.27))))
-    (property "LCSC" "C2861750"
+    (property "Datasheet" "https://www.ti.com/lit/ds/symlink/tlv767.pdf"
+      (at 335.28 40.64 0)
+      (hide yes)
+      (show_name no)
+      (do_not_autoplace no)
+      (effects
+        (font
+          (size 1.27 1.27))))
+    (property "Description" "1A 16V Low Dropout Voltage Regulator, Fixed Output 3.3V with SNS, WSON6 (TLV767, 18 V abs max VIN/EN)"
+      (at 335.28 40.64 0)
+      (hide yes)
+      (show_name no)
+      (do_not_autoplace no)
+      (effects
+        (font
+          (size 1.27 1.27))))
+    (property "MPN" "TI TLV76733DRVR"
+      (at 335.28 40.64 0)
+      (hide yes)
+      (show_name no)
+      (do_not_autoplace no)
+      (effects
+        (font
+          (size 1.27 1.27))))
+    (property "LCSC" "C2848334"
       (at 335.28 40.64 0)
       (hide yes)
@@
       (xy 342.9 38.1)
       (xy 345.44 38.1))
+    (stroke
+      (width 0)
+      (type default))
+)
+  (wire
+    (pts
+      (xy 342.9 40.64)
+      (xy 345.44 40.64))
     (stroke
       (width 0)
@@
           (reference "#PWR38")
           (unit 1)))))
+  (wire
+    (pts
+      (xy 345.44 38.1)
+      (xy 345.44 40.64))
+    (stroke
+      (width 0)
+      (type default))
+)
   (symbol
     (lib_id "power:+3.3V")

Commit message: JLC order fixes: LSM6DSV IMU, THT by JLC, one-line-per-part BOM, Gerber-frame CPL
Placing the first real JLCPCB Economic PCBA order for v1.3 turned up
problems that DRC and the review waves didn't catch. Copper is unchanged
(Gerbers regenerate identical apart from timestamps).

- U4: LSM6DSV16X (C5267406) -> LSM6DSV (C41785564). JLC lists the
  LSM6DSV16X as "Standard PCBA only" (X-ray); the LSM6DSV is allowed on
  Economic. Same LGA-14 pinout and I2C wiring, same registers for
  everything the firmware and SFLP use, WHO_AM_I 0x70. It lacks the MLC,
  Qvar and analog hub, none of which the board uses. Project symbol
  renamed; board/schematic fields updated (DRC parity 0).
- J1/J3 get LCSC C5383109 (HanElectricity 2541WV-2x10P) and J1-J3 are
  assembled by JLC instead of hand-soldered.
- fab.sh BOM: grouped by LCSC number, so JLC no longer unselects
  R1/R8/R10, R4/R5, R7/R9/R11 and SW1/SW2 as "multiple lines matched to
  the same part"; THT parts included.
- fab.sh CPL: written in the Gerber frame (JLC flagged every part as
  offset from the board with the old lower-left origin); rotation and
  origin corrections keyed by LCSC part, including the header (-90,
  centred) and USB4085 origin; asserts every part lands on the board.
- Docs: README (IMU, ordering: ENIG needs green on Economic, avoid black
  mask for the 0.11 mm USB-C pad gaps), REVIEW.md "JLC order round",
  parts/IMU research, firmware strings. Renode tests 10/10.

Co-Authored-By: Claude Opus 5.5 <noreply@anthropic.com>
Claude-Session: https://claude.ai/code/session_017LucoBJmh2YFvzHpYSamwe
Parts:
- J1, J3: LCSC (none) -> C5383109; MPN (none) -> HanElectricity 2541WV-2x10P (male, 6 mm pins, 3 mm tail)
- U4: value LSM6DSV16X -> LSM6DSV; symbol nicklink:LSM6DSV16X -> nicklink:LSM6DSV; LCSC C5267406 -> C41785564; MPN ST LSM6DSV16XTR -> ST LSM6DSV (JLC: LSM6DSVETR)
Changed lines of the file:
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@@
+        (font
+          (size 1.27 1.27))))
+    (property "MPN" "HanElectricity 2541WV-2x10P (male, 6 mm pins, 3 mm tail)"
+      (at 299.72 139.7 0)
+      (hide yes)
+      (show_name no)
+      (do_not_autoplace no)
+      (effects
+        (font
+          (size 1.27 1.27))))
+    (property "LCSC" "C5383109"
+      (at 299.72 139.7 0)
+      (hide yes)
+      (show_name no)
+      (do_not_autoplace no)
+      (effects
         (font
           (size 1.27 1.27))))
@@
         (font
           (size 1.27 1.27))))
+    (property "MPN" "HanElectricity 2541WV-2x10P (male, 6 mm pins, 3 mm tail)"
+      (at 365.76 139.7 0)
+      (hide yes)
+      (show_name no)
+      (do_not_autoplace no)
+      (effects
+        (font
+          (size 1.27 1.27))))
+    (property "LCSC" "C5383109"
+      (at 365.76 139.7 0)
+      (hide yes)
+      (show_name no)
+      (do_not_autoplace no)
+      (effects
+        (font
+          (size 1.27 1.27))))
     (pin "1"
 )
@@
           (unit 1)))))
   (symbol
-    (lib_id "nicklink:LSM6DSV16X")
+    (lib_id "nicklink:LSM6DSV")
     (at 309.88 190.5 0)
     (unit 1)
@@
           (size 1.27 1.27))
         (justify left)))
-    (property "Value" "LSM6DSV16X"
+    (property "Value" "LSM6DSV"
       (at 298.45 177.8 0)
       (show_name no)
@@
         (font
           (size 1.27 1.27))))
-    (property "Datasheet" "https://www.st.com/resource/en/datasheet/lsm6dsv16x.pdf"
+    (property "Datasheet" "https://www.st.com/resource/en/datasheet/lsm6dsv.pdf"
       (at 309.88 190.5 0)
       (hide yes)
@@
         (font
           (size 1.27 1.27))))
-    (property "MPN" "ST LSM6DSV16XTR"
+    (property "MPN" "ST LSM6DSV (JLC: LSM6DSVETR)"
       (at 309.88 190.5 0)
       (hide yes)
@@
         (font
           (size 1.27 1.27))))
-    (property "LCSC" "C5267406"
+    (property "LCSC" "C41785564"
       (at 309.88 190.5 0)
       (hide yes)
